File: Quilter.kicad_sch (KiCad schematic)
At the start: 30 parts, among them J1 Eurorack_10_pin_power, J2 Conn_01x08_Male, J3 Conn_01x08_Male, J4 IO, U1 TL072, U2 TL074

Commit message: First draft of component PCB routed
Parts:
- added C37, C38: 1uF, Capacitor_SMD:C_0603_1608Metric_Pad1.08x0.95mm_HandSolder, symbol Device:C_Small
- J2, J3: footprint Connector_PinHeader_2.54mm:PinHeader_1x08_P2.54mm_Vertical -> Connector_PinHeader_2.54mm:PinHeader_1x10_P2.54mm_Vertical; symbol Connector:Conn_01x08_Male -> Connector:Conn_01x10_Male
- J4: footprint Connector_PinHeader_2.54mm:PinHeader_1x06_P2.54mm_Vertical -> Connector_PinHeader_2.54mm:PinHeader_1x10_P2.54mm_Vertical; symbol Connector:Conn_01x06_Male -> Connector:Conn_01x10_Male
Connections:
- net -12V: now also U2.11 (V-), C37.1, C38.1
- net AUDIO_BUFF1: now also J2.5 (Pin_5); no longer J2.4 (Pin_4)
- net AUDIO_BUFF2: now also J3.3 (Pin_3), R14.1, U2.14; no longer J3.4 (Pin_4), R12.1, U2.7
- net AUDIO_BUFF3: now also J3.2 (Pin_2), R12.1, U2.7; no longer J3.6 (Pin_6), R13.1, U2.8
- net AUDIO_BUFF4: now also J2.8 (Pin_8), R13.1, U2.8; no longer J3.8 (Pin_8), R14.1, U2.14
- net AUDIO_IN1: now also J2.10 (Pin_10); no longer J2.1 (Pin_1)
- net AUDIO_IN2: now also J3.9 (Pin_9); no longer J3.1 (Pin_1)
- net AUDIO_IN3: now also J4.9 (Pin_9); no longer J2.6 (Pin_6)
- net AUDIO_IN4: now also J4.5 (Pin_5); no longer J3.7 (Pin_7)
- net AUDIO_MIX: now also J2.9 (Pin_9); no longer J4.6 (Pin_6)
- net Audio_Out2: now also R10.2; no longer R8.2
- net Audio_Out3: now also R8.2; no longer R9.2
- net Audio_Out4: now also R9.2; no longer R10.2
- net FREQ_CV1: now also J4.6 (Pin_6); no longer J2.2 (Pin_2)
- net FREQ_CV2: now also J3.8 (Pin_8); no longer J3.2 (Pin_2)
- net FREQ_CV3: now also J4.8 (Pin_8); no longer J2.7 (Pin_7)
- net FREQ_CV4: now also J4.3 (Pin_3); no longer J4.1 (Pin_1)
- net FREQ_POT: now also J4.7 (Pin_7); no longer J4.3 (Pin_3)
- net FREQ_POT_5V: now also J3.10 (Pin_10); no longer J4.5 (Pin_5)
- net FREQ_V_OCT1: now also J2.4 (Pin_4); no longer J2.3 (Pin_3)
- net FREQ_V_OCT2: now also J3.4 (Pin_4); no longer J3.3 (Pin_3)
- net FREQ_V_OCT3: now also J4.10 (Pin_10); no longer J2.8 (Pin_8)
- net GND: now also J2.6 (Pin_6), J3.6 (Pin_6), C37.2, C38.2; no longer J2.5 (Pin_5), J3.5 (Pin_5), U2.11 (V-)

Commit message: Started Controls PCB
Parts:
- J1: renamed from J2; value Conn_01x08_Male -> Conn_01x10_Male
- J2: renamed from J3; value Conn_01x08_Male -> Conn_01x10_Male
- J3: renamed from J4; value IO -> Conn_01x10_Male
- renumbered C37 to C5, C38 to C8, J1 to J4
Changed lines of the file:
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@@
   (symbol (lib_id "Connector:Conn_01x10_Male") (at 83.185 130.175 0) (unit 1)
     (in_bom yes) (on_board yes) (fields_autoplaced)
-    (property "Reference" "J3" (id 0) (at 83.82 114.3 0))
-    (property "Value" "Conn_01x08_Male" (id 1) (at 83.82 116.84 0))
+    (property "Reference" "J2" (id 0) (at 83.82 114.3 0))
+    (property "Value" "Conn_01x10_Male" (id 1) (at 83.82 116.84 0))
     (property "Footprint" "Connector_PinHeader_2.54mm:PinHeader_1x10_P2.54mm_Vertical" (id 2) (at 83.185 130.175 0)
       (effects (font (size 1.27 1.27)) hide)
@@
   (symbol (lib_id "Device:C_Small") (at 121.285 182.88 90) (unit 1)
     (in_bom yes) (on_board yes)
-    (property "Reference" "C38" (id 0) (at 121.285 186.69 90))
+    (property "Reference" "C8" (id 0) (at 121.285 186.69 90))
     (property "Value" "1uF" (id 1) (at 121.2913 179.07 90))
     (property "Footprint" "Capacitor_SMD:C_0603_1608Metric_Pad1.08x0.95mm_HandSolder" (id 2) (at 121.285 182.88 0)
@@
   (symbol (lib_id "Connector:Conn_01x10_Male") (at 82.55 95.885 0) (unit 1)
     (in_bom yes) (on_board yes) (fields_autoplaced)
-    (property "Reference" "J2" (id 0) (at 83.185 80.01 0))
-    (property "Value" "Conn_01x08_Male" (id 1) (at 83.185 82.55 0))
+    (property "Reference" "J1" (id 0) (at 83.185 80.01 0))
+    (property "Value" "Conn_01x10_Male" (id 1) (at 83.185 82.55 0))
     (property "Footprint" "Connector_PinHeader_2.54mm:PinHeader_1x10_P2.54mm_Vertical" (id 2) (at 82.55 95.885 0)
       (effects (font (size 1.27 1.27)) hide)
@@
   (symbol (lib_id "Eurorack_Header:Eurorack_10_pin_power") (at 43.815 172.085 180) (unit 1)
     (in_bom yes) (on_board yes)
-    (property "Reference" "J1" (id 0) (at 38.735 179.705 0))
+    (property "Reference" "J4" (id 0) (at 38.735 179.705 0))
     (property "Value" "Eurorack_10_pin_power" (id 1) (at 37.465 163.195 0))
     (property "Footprint" "Custom_Footprints:Eurorack_10_pin_header" (id 2) (at 43.815 172.085 0)
@@
   (symbol (lib_id "Device:C_Small") (at 100.33 182.88 90) (unit 1)
     (in_bom yes) (on_board yes)
-    (property "Reference" "C37" (id 0) (at 100.33 186.69 90))
+    (property "Reference" "C5" (id 0) (at 100.33 186.69 90))
     (property "Value" "1uF" (id 1) (at 100.3363 179.07 90))
     (property "Footprint" "Capacitor_SMD:C_0603_1608Metric_Pad1.08x0.95mm_HandSolder" (id 2) (at 100.33 182.88 0)
@@
   (symbol (lib_id "Connector:Conn_01x10_Male") (at 114.935 112.395 0) (unit 1)
     (in_bom yes) (on_board yes) (fields_autoplaced)
-    (property "Reference" "J4" (id 0) (at 115.57 96.52 0))
-    (property "Value" "IO" (id 1) (at 115.57 99.06 0))
+    (property "Reference" "J3" (id 0) (at 115.57 96.52 0))
+    (property "Value" "Conn_01x10_Male" (id 1) (at 115.57 99.06 0))
     (property "Footprint" "Connector_PinHeader_2.54mm:PinHeader_1x10_P2.54mm_Vertical" (id 2) (at 114.935 112.395 0)
       (effects (font (size 1.27 1.27)) hide)
@@
       (reference "C4") (unit 1) (value "1uF") (footprint "Capacitor_SMD:C_0603_1608Metric_Pad1.08x0.95mm_HandSolder")
     )
-    (path "/e84f8fd9-bd0a-4839-99bd-bd22e1164470/4f532a1f-7ffe-4156-9778-aee108f260cb"
-      (reference "C5") (unit 1) (value "3.3nF") (footprint "Capacitor_SMD:C_0603_1608Metric_Pad1.08x0.95mm_HandSolder")
+    (path "/a8b528a7-dda2-4a2b-b4fc-21c8234268be"
+      (reference "C5") (unit 1) (value "1uF") (footprint "Capacitor_SMD:C_0603_1608Metric_Pad1.08x0.95mm_HandSolder")
     )
     (path "/e84f8fd9-bd0a-4839-99bd-bd22e1164470/a82fa926-487a-4c80-8cd3-f96c4eea9485"
@@
       (reference "C7") (unit 1) (value "6.8nF") (footprint "Capacitor_SMD:C_0603_1608Metric_Pad1.08x0.95mm_HandSolder")
     )
-    (path "/e84f8fd9-bd0a-4839-99bd-bd22e1164470/1d87cdf4-4f83-47cf-81a5-94f0703716a0"
-      (reference "C8") (unit 1) (value "6.8nF") (footprint "Capacitor_SMD:C_0603_1608Metric_Pad1.08x0.95mm_HandSolder")
+    (path "/71e78113-df27-4c0c-8d84-46bb2b1169a8"
+      (reference "C8") (unit 1) (value "1uF") (footprint "Capacitor_SMD:C_0603_1608Metric_Pad1.08x0.95mm_HandSolder")
     )
     (path "/e84f8fd9-bd0a-4839-99bd-bd22e1164470/9f668a87-19d4-4d7b-b3ff-e6f382f127f3"
@@
       (reference "C36") (unit 1) (value "1uF") (footprint "Capacitor_SMD:C_0603_1608Metric_Pad1.08x0.95mm_HandSolder")
     )
-    (path "/a8b528a7-dda2-4a2b-b4fc-21c8234268be"
-      (reference "C37") (unit 1) (value "1uF") (footprint "Capacitor_SMD:C_0603_1608Metric_Pad1.08x0.95mm_HandSolder")
-    )
-    (path "/71e78113-df27-4c0c-8d84-46bb2b1169a8"
-      (reference "C38") (unit 1) (value "1uF") (footprint "Capacitor_SMD:C_0603_1608Metric_Pad1.08x0.95mm_HandSolder")
+    (path "/e84f8fd9-bd0a-4839-99bd-bd22e1164470/4f532a1f-7ffe-4156-9778-aee108f260cb"
+      (reference "C37") (unit 1) (value "3.3nF") (footprint "Capacitor_SMD:C_0603_1608Metric_Pad1.08x0.95mm_HandSolder")
+    )
+    (path "/e84f8fd9-bd0a-4839-99bd-bd22e1164470/1d87cdf4-4f83-47cf-81a5-94f0703716a0"
+      (reference "C38") (unit 1) (value "6.8nF") (footprint "Capacitor_SMD:C_0603_1608Metric_Pad1.08x0.95mm_HandSolder")
     )
     (path "/e84f8fd9-bd0a-4839-99bd-bd22e1164470/60546b12-55d9-4ab4-9cd7-c432a53568d2"
@@
       (reference "FREQ_OFFSET4") (unit 1) (value "50k") (footprint "Potentiometer_SMD:Potentiometer_Bourns_TC33X_Vertical")
     )
+    (path "/8efaa33f-ca82-4e3b-8b28-d24d5dd94ed9"
+      (reference "J1") (unit 1) (value "Conn_01x10_Male") (footprint "Connector_PinHeader_2.54mm:PinHeader_1x10_P2.54mm_Vertical")
+    )
+    (path "/3c593478-0576-4e30-bad8-fa652ed5b16d"
+      (reference "J2") (unit 1) (value "Conn_01x10_Male") (footprint "Connector_PinHeader_2.54mm:PinHeader_1x10_P2.54mm_Vertical")
+    )
+    (path "/dd85f030-493f-4501-9a8a-e07928a49b79"
+      (reference "J3") (unit 1) (value "Conn_01x10_Male") (footprint "Connector_PinHeader_2.54mm:PinHeader_1x10_P2.54mm_Vertical")
+    )
     (path "/8f085082-4aeb-402b-b84f-d7f4cac09e17"
-      (reference "J1") (unit 1) (value "Eurorack_10_pin_power") (footprint "Custom_Footprints:Eurorack_10_pin_header")
-    )
-    (path "/8efaa33f-ca82-4e3b-8b28-d24d5dd94ed9"
-      (reference "J2") (unit 1) (value "Conn_01x08_Male") (footprint "Connector_PinHeader_2.54mm:PinHeader_1x10_P2.54mm_Vertical")
-    )
-    (path "/3c593478-0576-4e30-bad8-fa652ed5b16d"
-      (reference "J3") (unit 1) (value "Conn_01x08_Male") (footprint "Connector_PinHeader_2.54mm:PinHeader_1x10_P2.54mm_Vertical")
-    )
-    (path "/dd85f030-493f-4501-9a8a-e07928a49b79"
-      (reference "J4") (unit 1) (value "IO") (footprint "Connector_PinHeader_2.54mm:PinHeader_1x10_P2.54mm_Vertical")
+      (reference "J4") (unit 1) (value "Eurorack_10_pin_power") (footprint "Custom_Footprints:Eurorack_10_pin_header")
     )
     (path "/d0e40d50-e24f-4dca-95c7-4f1817993833"
