File: Quilter_Controls.kicad_sch (KiCad schematic)
At the start: 14 parts

Commit message: Started Controls PCB
Parts:
- removed J? (x2): Conn_01x08_Male, Connector_PinHeader_2.54mm:PinHeader_1x08_P2.54mm_Vertical, symbol Connector:Conn_01x08_Male
- removed J?: IO, Connector_PinHeader_2.54mm:PinHeader_1x06_P2.54mm_Vertical, symbol Connector:Conn_01x06_Male
- added J1, J2, J3: Conn_01x10_Male, Connector_PinHeader_2.54mm:PinHeader_1x10_P2.54mm_Vertical, symbol Connector:Conn_01x10_Male
- added J10: Conn_01x04_Male, Connector_PinHeader_2.54mm:PinHeader_1x04_P2.54mm_Vertical, symbol Connector:Conn_01x04_Male
- added J9: Conn_02x04_Top_Bottom, Connector_PinHeader_2.54mm:PinHeader_2x04_P2.54mm_Vertical, symbol Connector_Generic:Conn_02x04_Top_Bottom
- gave numbers to parts that had none: 10
Connections:
- net AUDIO_BUFF1: now also J1.5 (Pin_5), J10.1 (Pin_1)
- net AUDIO_BUFF2: now also J10.2 (Pin_2), J2.3 (Pin_3)
- net AUDIO_BUFF3: now also J10.3 (Pin_3), J2.2 (Pin_2)
- net AUDIO_BUFF4: now also J1.8 (Pin_8), J10.4 (Pin_4)
- net AUDIO_IN1: now also J1.10 (Pin_10), J9.1 (Pin_1)
- net AUDIO_IN2: now also J2.9 (Pin_9), J9.2 (Pin_2)
- net AUDIO_IN3: now also J3.9 (Pin_9), J9.3 (Pin_3)
- net AUDIO_IN4: now also J3.5 (Pin_5), J9.4 (Pin_4)
- net AUDIO_MIX: now also J1.9 (Pin_9)
- net FREQ_CV1: now also J3.6 (Pin_6)
- net FREQ_CV2: now also J2.8 (Pin_8)
- net FREQ_CV3: now also J3.8 (Pin_8)
- net FREQ_CV4: now also J3.3 (Pin_3)
- net FREQ_POT: now also J3.7 (Pin_7)
- net FREQ_POT_5V: now also J2.10 (Pin_10)
- net FREQ_V_OCT1: now also J1.4 (Pin_4), J9.5 (Pin_5)
- net FREQ_V_OCT2: now also J2.4 (Pin_4), J9.6 (Pin_6)
- net FREQ_V_OCT3: now also J3.10 (Pin_10), J9.7 (Pin_7)
- net FREQ_V_OCT4: now also J3.2 (Pin_2), J9.8 (Pin_8)
- net GND: now also J1.6 (Pin_6), J2.6 (Pin_6)
- net Q_POT: now also J3.4 (Pin_4)

Commit message: First draft routing of Controls PCB
Parts:
- J9: symbol Connector_Generic:Conn_02x04_Top_Bottom -> Connector_Generic:Conn_02x04_Odd_Even
Connections:
- net +12V: now also J2.1 (Pin_1)
- net -12V: now also J1.1 (Pin_1)
- net AUDIO_BUFF3: now also J1.3 (Pin_3); no longer J2.2 (Pin_2)
- net AUDIO_BUFF4: now also J2.5 (Pin_5); no longer J1.8 (Pin_8)
- net AUDIO_IN2: now also J2.10 (Pin_10), J9.3 (Pin_3); no longer J2.9 (Pin_9), J9.2 (Pin_2)
- net AUDIO_IN3: now also J9.5 (Pin_5); no longer J9.3 (Pin_3)
- net AUDIO_IN4: now also J3.1 (Pin_1), J9.7 (Pin_7); no longer J3.5 (Pin_5), J9.4 (Pin_4)
- net FREQ_CV1: now also J3.7 (Pin_7); no longer J3.6 (Pin_6)
- net FREQ_CV4: now also J3.6 (Pin_6); no longer J3.3 (Pin_3)
- net FREQ_POT: now also J3.5 (Pin_5); no longer J3.7 (Pin_7)
- net FREQ_POT_5V: now also J2.7 (Pin_7); no longer J2.10 (Pin_10)
- net FREQ_V_OCT1: now also J9.2 (Pin_2); no longer J9.5 (Pin_5)
- net FREQ_V_OCT2: now also J1.7 (Pin_7), J9.4 (Pin_4); no longer J2.4 (Pin_4), J9.6 (Pin_6)
- net FREQ_V_OCT3: now also J9.6 (Pin_6); no longer J9.7 (Pin_7)
Other:
- moved on the sheet: J1, J2, J3
