File: Quilter_Components.kicad_pcb (KiCad board)
At the start: 4 copper layers, 40.4 x 100 mm, 160 parts, among them J1 Conn_01x10_Male, J2 Conn_01x10_Male, J3 Conn_01x10_Male, J4 Eurorack_10_pin_power, U1 TL072, U10 SSI2144, U2 TL074, U3 TL074, U4 TL074, U5 SSI2144, U7 SSI2144, U9 SSI2144

Commit message: Prepared v2 Controls and Components for manufacture
Parts:
- C11, C19, C27, C35: value 10nF_C0G -> 10nF
Changed lines of the file:
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@@
     (descr "SOD-123")
     (tags "SOD-123")
-    (property "Part_Number" "C8598")
+    (property "Part_Number" "")
     (property "Sheetfile" "Quilter_Components.kicad_sch")
     (property "Sheetname" "")
@@
     (descr "Resistor SMD 0603 (1608 Metric), square (rectangular) end terminal, IPC_7351 nominal with elongated pad for handsoldering. (Body size source: IPC-SM-782 page 72, https://www.pcb-3d.com/wordpress/wp-content/uploads/ipc-sm-782a_amendment_1_and_2.pdf), generated with kicad-footprint-generator")
     (tags "resistor handsolder")
-    (property "Part_Number" "C25804")
+    (property "Part_Number" "")
     (property "Sheetfile" "Quilter_Components.kicad_sch")
     (property "Sheetname" "")
@@
       (effects (font (size 1 1) (thickness 0.15)))
     )
-    (fp_text value "10nF_C0G" (at 0 1.43) (layer "F.Fab")
+    (fp_text value "10nF" (at 0 1.43) (layer "F.Fab")
       (effects (font (size 1 1) (thickness 0.15)))
     )
@@
     (descr "Resistor SMD 0603 (1608 Metric), square (rectangular) end terminal, IPC_7351 nominal with elongated pad for handsoldering. (Body size source: IPC-SM-782 page 72, https://www.pcb-3d.com/wordpress/wp-content/uploads/ipc-sm-782a_amendment_1_and_2.pdf), generated with kicad-footprint-generator")
     (tags "resistor handsolder")
-    (property "Part_Number" "C25804")
+    (property "Part_Number" "")
     (property "Sheetfile" "Quilter_Components.kicad_sch")
     (property "Sheetname" "")
@@
     (descr "Resistor SMD 0603 (1608 Metric), square (rectangular) end terminal, IPC_7351 nominal with elongated pad for handsoldering. (Body size source: IPC-SM-782 page 72, https://www.pcb-3d.com/wordpress/wp-content/uploads/ipc-sm-782a_amendment_1_and_2.pdf), generated with kicad-footprint-generator")
     (tags "resistor handsolder")
-    (property "Part_Number" "C25804")
+    (property "Part_Number" "")
     (property "Sheetfile" "Quilter_Components.kicad_sch")
     (property "Sheetname" "")
@@
     (descr "SMD capacitor, aluminum electrolytic, Panasonic, 4.0x5.8mm")
     (tags "capacitor electrolytic")
-    (property "Part_Number" "C134793")
-    (property "Rotation" "270")
+    (property "Part_Number" "")
+    (property "Rotation" "")
     (property "Sheetfile" "Quilter_Components.kicad_sch")
     (property "Sheetname" "")
@@
       (effects (font (size 1 1) (thickness 0.15)))
     )
-    (fp_text value "10nF_C0G" (at 0 1.43) (layer "F.Fab")
+    (fp_text value "10nF" (at 0 1.43) (layer "F.Fab")
       (effects (font (size 1 1) (thickness 0.15)))
     )
@@
     (property "Sheetfile" "Quilter_Components.kicad_sch")
     (property "Sheetname" "")
+    (property "exclude_from_bom" "")
     (attr exclude_from_pos_files exclude_from_bom)
     (fp_text reference "TP2" (at 0 -2.75) (layer "F.SilkS") hide
@@
     (descr "Resistor SMD 0603 (1608 Metric), square (rectangular) end terminal, IPC_7351 nominal with elongated pad for handsoldering. (Body size source: IPC-SM-782 page 72, https://www.pcb-3d.com/wordpress/wp-content/uploads/ipc-sm-782a_amendment_1_and_2.pdf), generated with kicad-footprint-generator")
     (tags "resistor handsolder")
-    (property "Part_Number" "C25804")
+    (property "Part_Number" "")
     (property "Sheetfile" "Quilter_Components.kicad_sch")
     (property "Sheetname" "")
@@
     (descr "SOD-123")
     (tags "SOD-123")
-    (property "Part_Number" "C8598")
+    (property "Part_Number" "")
     (property "Sheetfile" "Quilter_Components.kicad_sch")
     (property "Sheetname" "")
@@
     (descr "Resistor SMD 0603 (1608 Metric), square (rectangular) end terminal, IPC_7351 nominal with elongated pad for handsoldering. (Body size source: IPC-SM-782 page 72, https://www.pcb-3d.com/wordpress/wp-content/uploads/ipc-sm-782a_amendment_1_and_2.pdf), generated with kicad-footprint-generator")
     (tags "resistor handsolder")
-    (property "Part_Number" "C25804")
+    (property "Part_Number" "")
     (property "Sheetfile" "Quilter_Components.kicad_sch")
     (property "Sheetname" "")
@@
     (descr "Resistor SMD 0603 (1608 Metric), square (rectangular) end terminal, IPC_7351 nominal with elongated pad for handsoldering. (Body size source: IPC-SM-782 page 72, https://www.pcb-3d.com/wordpress/wp-content/uploads/ipc-sm-782a_amendment_1_and_2.pdf), generated with kicad-footprint-generator")
     (tags "resistor handsolder")
-    (property "Part_Number" "C25804")
+    (property "Part_Number" "")
     (property "Sheetfile" "Quilter_Components.kicad_sch")
     (property "Sheetname" "")
@@
     (descr "Resistor SMD 0603 (1608 Metric), square (rectangular) end terminal, IPC_7351 nominal with elongated pad for handsoldering. (Body size source: IPC-SM-782 page 72, https://www.pcb-3d.com/wordpress/wp-content/uploads/ipc-sm-782a_amendment_1_and_2.pdf), generated with kicad-footprint-generator")
     (tags "resistor handsolder")
-    (property "Part_Number" "C25804")
+    (property "Part_Number" "")
     (property "Sheetfile" "Quilter_Components.kicad_sch")
     (property "Sheetname" "")
@@
     (descr "Resistor SMD 0603 (1608 Metric), square (rectangular) end terminal, IPC_7351 nominal with elongated pad for handsoldering. (Body size source: IPC-SM-782 page 72, https://www.pcb-3d.com/wordpress/wp-content/uploads/ipc-sm-782a_amendment_1_and_2.pdf), generated with kicad-footprint-generator")
     (tags "resistor handsolder")
-    (property "Part_Number" "C25804")
+    (property "Part_Number" "")
     (property "Sheetfile" "Quilter_Components.kicad_sch")
     (property "Sheetname" "")
@@
     (descr "Resistor SMD 0603 (1608 Metric), square (rectangular) end terminal, IPC_7351 nominal with elongated pad for handsoldering. (Body size source: IPC-SM-782 page 72, https://www.pcb-3d.com/wordpress/wp-content/uploads/ipc-sm-782a_amendment_1_and_2.pdf), generated with kicad-footprint-generator")
     (tags "resistor handsolder")
-    (property "Part_Number" "C25804")
+    (property "Part_Number" "")
     (property "Sheetfile" "Quilter_Components.kicad_sch")
     (property "Sheetname" "")
@@
       (effects (font (size 1 1) (thickness 0.15)))
     )
-    (fp_text value "10nF_C0G" (at 0 1.43) (layer "F.Fab")
+    (fp_text value "10nF" (at 0 1.43) (layer "F.Fab")
       (effects (font (size 1 1) (thickness 0.15)))
     )
@@
     (property "Sheetfile" "Quilter_Components.kicad_sch")
     (property "Sheetname" "")
+    (property "exclude_from_bom" "")
     (attr exclude_from_pos_files exclude_from_bom)
     (fp_text reference "TP4" (at 0 -2.75) (layer "F.SilkS") hide
@@
     (descr "Resistor SMD 0603 (1608 Metric), square (rectangular) end terminal, IPC_7351 nominal with elongated pad for handsoldering. (Body size source: IPC-SM-782 page 72, https://www.pcb-3d.com/wordpress/wp-content/uploads/ipc-sm-782a_amendment_1_and_2.pdf), generated with kicad-footprint-generator")
     (tags "resistor handsolder")
-    (property "Part_Number" "C25804")
+    (property "Part_Number" "")
     (property "Sheetfile" "Quilter_Components.kicad_sch")
     (property "Sheetname" "")
@@
     (descr "Resistor SMD 0603 (1608 Metric), square (rectangular) end terminal, IPC_7351 nominal with elongated pad for handsoldering. (Body size source: IPC-SM-782 page 72, https://www.pcb-3d.com/wordpress/wp-content/uploads/ipc-sm-782a_amendment_1_and_2.pdf), generated with kicad-footprint-generator")
     (tags "resistor handsolder")
-    (property "Part_Number" "C25804")
+    (property "Part_Number" "")
     (property "Sheetfile" "Quilter_Components.kicad_sch")
     (property "Sheetname" "")
@@
     (property "Sheetfile" "Quilter_Components.kicad_sch")
     (property "Sheetname" "")
+    (property "exclude_from_bom" "")
     (attr exclude_from_pos_files exclude_from_bom)
     (fp_text reference "TP1" (at 0 -2.75) (layer "F.SilkS") hide
@@
     (descr "SMD capacitor, aluminum electrolytic, Panasonic, 4.0x5.8mm")
     (tags "capacitor electrolytic")
-    (property "Part_Number" "C134798")
-    (property "Rotation" "360")
+    (property "Part_Number" "")
+    (property "Rotation" "")
     (property "Sheetfile" "Quilter_Components.kicad_sch")
     (property "Sheetname" "")
@@
     (descr "Resistor SMD 0603 (1608 Metric), square (rectangular) end terminal, IPC_7351 nominal with elongated pad for handsoldering. (Body size source: IPC-SM-782 page 72, https://www.pcb-3d.com/wordpress/wp-content/uploads/ipc-sm-782a_amendment_1_and_2.pdf), generated with kicad-footprint-generator")
     (tags "resistor handsolder")
-    (property "Part_Number" "C25804")
+    (property "Part_Number" "")
     (property "Sheetfile" "Quilter_Components.kicad_sch")
     (property "Sheetname" "")
@@
     (descr "Resistor SMD 0603 (1608 Metric), square (rectangular) end terminal, IPC_7351 nominal with elongated pad for handsoldering. (Body size source: IPC-SM-782 page 72, https://www.pcb-3d.com/wordpress/wp-content/uploads/ipc-sm-782a_amendment_1_and_2.pdf), generated with kicad-footprint-generator")
     (tags "resistor handsolder")
-    (property "Part_Number" "C25804")
+    (property "Part_Number" "")
     (property "Sheetfile" "Quilter_Components.kicad_sch")
     (property "Sheetname" "")
@@
     (property "Sheetfile" "Quilter_Components.kicad_sch")
     (property "Sheetname" "")
+    (property "exclude_from_bom" "")
     (attr exclude_from_pos_files exclude_from_bom)
     (fp_text reference "TP3" (at 0 -2.75) (layer "F.SilkS") hide
@@
       (effects (font (size 1 1) (thickness 0.15)))
     )
-    (fp_text value "10nF_C0G" (at 0 1.43) (layer "F.Fab")
+    (fp_text value "10nF" (at 0 1.43) (layer "F.Fab")
       (effects (font (size 1 1) (thickness 0.15)))
     )
