File: HP10/Filter_Voice.kicad_sch (KiCad schematic)
At the start: 26 parts, among them U3 TL074, U5 SSI2144

Commit message: Started layout for 8HP alternative
Parts:
- removed U3: TL074, Package_SO:SOIC-14_3.9x8.7mm_P1.27mm, symbol Amplifier_Operational:TL074
- added C39: 1uF, Capacitor_SMD:C_0603_1608Metric_Pad1.08x0.95mm_HandSolder, symbol Device:C_Small
- added U3: TL072, Package_SO:SO-8_3.9x4.9mm_P1.27mm, symbol Amplifier_Operational:TL072
- renumbered U5 to U4
Connections:
- net +12V: now also C12.1, U3.8 (V+)
- net -12V: now also C39.1, U3.4 (V-); no longer C12.2
- net AUDIO_OUT: now also U3.7
- net GND: now also C12.2, C39.2, U3.3 (+), U3.5 (+); no longer C12.1
- net at R18.1, R19.1, R20.1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: now also U3.2 (-)
- net at C10.2, R25.2, U4.3 (OUT): now also U3.6 (-)
- net at R22.2, V_OCT1.2, V_OCT1.3: now also U3.1
